File: hardware/mainBoard/DC_DCs.sch (KiCad schematic (older format))
At the start: 30 parts

Commit message: Added the power part of the schematic
Parts:
- U?: symbol chinaland:SGM3204 -> prockeckv2-rescue:SGM3204-chinaland
- U?: symbol chinaland:HX3242 -> prockeckv2-rescue:HX3242-chinaland
- U?: symbol chinaland:HX3001 -> prockeckv2-rescue:HX3001-chinaland
Changed lines of the file:
@@
 EESchema Schematic File Version 4
 LIBS:prockeckv2-cache
-LIBS:forcenOne-cache
-EELAYER 26 0
+EELAYER 30 0
 EELAYER END
 $Descr A4 11693 8268
@@
 $EndDescr
 $Comp
-L chinaland:SGM3204 U?
+L prockeckv2-rescue:SGM3204-chinaland U?
 U 1 1 5E85D6AB
 P 2500 1300
@@
 Vbatt
 $Comp
-L chinaland:HX3242 U?
+L prockeckv2-rescue:HX3242-chinaland U?
 U 1 1 5E87EE6B
 P 9000 1450
@@
 SENSOR_EN
 $Comp
-L chinaland:HX3001 U?
+L prockeckv2-rescue:HX3001-chinaland U?
 U 1 1 5E886D9C
 P 5250 1450
