File: hardware/mainBoard/Peripherals.sch (KiCad schematic (older format))
At the start: 0 parts

Commit message: Added external connections, analog conditioning and several items
Parts:
- added J?: MicroSD, symbol Chinaland:MicroSD
- added J?: Conn_01x06_Male, symbol Connector:Conn_01x06_Male
- added U?: E19-868M30S, symbol Chinaland:E19-868M30S
- added U?: W25Q64JV, symbol Chinaland:W25Q64JV
Connections:
- new net +3V3: J?.1 (Pin_1), J?.4 (VDD), U?.8 (VCC)
- new net +5V: U?.11 (VCC)
- new net GND: J?.10 (SHIELD), J?.2 (Pin_2), J?.6 (VSS), U?.1 (GND), U?.10 (GND), U?.18 (GND), U?.20 (GND), U?.21 (GND), U?.22 (GND), U?.4 (GND), U?.9 (GND)
- new net IO2_1: U?.1 (~CS)
- new net IO2_10: J?.3 (Pin_3)
- new net IO2_11: J?.5 (Pin_5)
- new net IO2_2: U?.8 (RST)
- new net IO2_3: U?.15 (~SS)
- new net IO2_4: U?.7 (DIO0)
- new net IO2_5: U?.6 (DIO1)
- new net IO2_6: U?.5 (DIO2)
- new net IO2_7: U?.4 (DIO3)
- new net IO2_8: U?.16 (TXEN)
- new net IO2_9: U?.17 (RXEN)
- new net SDIO_CK: J?.5 (CLK)
- new net SDIO_CMD: J?.3 (CMD)
- new net SDIO_D0: J?.7 (DAT0)
- new net SDIO_D1: J?.8 (DAT1)
- new net SDIO_D2: J?.1 (DAT2)
- new net SDIO_D3: J?.2 (DAT3/CD)
- new net SPI1_MISO: U?.13 (MISO), U?.2 (DO)
- new net SPI1_MOSI: J?.4 (Pin_4), U?.14 (MOSI), U?.5 (DI)
- new net SPI1_SCK: J?.6 (Pin_6), U?.12 (SCK), U?.6 (CLK)
- no-connect marks 0 -> 5
