File: hardware/mainBoard/Controlled Power.sch (KiCad schematic (older format))
At the start: 22 parts, among them J21 Screw_Terminal_01x02, J22 Screw_Terminal_01x02, J23 Screw_Terminal_01x02, J24 Screw_Terminal_01x02, Q4 S8050, Q5 S8050, Q6 AO3415, Q7 AO3415, Q8 AP2300, Q9 AP2300

Commit message: First working software
Parts:
- F1, F2, F3, F4: URL (none) -> https://lcsc.com/product-detail/PTC-Resettable-Fuses_TECHFU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
- J21, J22, J23, J24: footprint TerminalBlock:TerminalBlock_bornier-2_P5.08mm -> Connector_PinHeader_2.54mm:PinHeader_1x02_P2.54mm_Vertical
- Q4, Q5: URL (none) -> https://lcsc.com/product-detail/Transistors-NPN-PNP_S8050_C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
- Q6, Q7: URL (none) -> https://lcsc.com/product-detail/MOSFET_Alpha-Omega-Semicon_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
- Q8, Q9: URL (none) -> https://lcsc.com/product-detail/MOSFET_ALLPOWER-ShenZhen-Qu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
- R59, R60, R61, R62, R65, R66: URL (none) -> https://lcsc.com/product-detail/Chip-Resistor-Surface-Mount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
- R63, R64: URL (none) -> https://lcsc.com/product-detail/New-Arrivals_SANYEAR-SY0603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
Changed lines of the file:
@@
 EESchema Schematic File Version 4
+LIBS:prockeckv2-cache
 EELAYER 30 0
 EELAYER END
@@
 F 2 "Resistor_SMD:R_0603_1608Metric_Pad1.05x0.95mm_HandSolder" V 3130 2900 50  0001 C CNN
 F 3 "~" H 3200 2900 50  0001 C CNN
+F 4 "https://lcsc.com/product-detail/Chip-Resistor-Surface-Mount_100KR-1003-1_C14675.html" H 3200 2900 50  0001 C CNN "URL"
 	1    3200 2900
 	0    1    1    0
@@
 F 2 "Resistor_SMD:R_0603_1608Metric_Pad1.05x0.95mm_HandSolder" V 3630 2450 50  0001 C CNN
 F 3 "~" H 3700 2450 50  0001 C CNN
+F 4 "https://lcsc.com/product-detail/Chip-Resistor-Surface-Mount_100KR-1003-1_C14675.html" H 3700 2450 50  0001 C CNN "URL"
 	1    3700 2450
 	-1   0    0    1
@@
 F 2 "Package_TO_SOT_SMD:SOT-23_Handsoldering" H 4800 2750 50  0001 C CNN
 F 3 "~" H 4600 2650 50  0001 C CNN
+F 4 "https://lcsc.com/product-detail/MOSFET_Alpha-Omega-Semicon_AO3415_Alpha-Omega-Semicon-AOS-AO3415_C14354.html" H 4600 2650 50  0001 C CNN "URL"
 	1    4600 2650
 	1    0    0    1
@@
 F 0 "J21" H 5030 2992 50  0000 L CNN
 F 1 "Screw_Terminal_01x02" H 5030 2901 50  0000 L CNN
-F 2 "TerminalBlock:TerminalBlock_bornier-2_P5.08mm" H 4950 3000 50  0001 C CNN
+F 2 "Connector_PinHeader_2.54mm:PinHeader_1x02_P2.54mm_Vertical" H 4950 3000 50  0001 C CNN
 F 3 "~" H 4950 3000 50  0001 C CNN
 	1    4950 3000
@@
 F 2 "Resistor_SMD:R_0603_1608Metric_Pad1.05x0.95mm_HandSolder" V 3130 4400 50  0001 C CNN
 F 3 "~" H 3200 4400 50  0001 C CNN
+F 4 "https://lcsc.com/product-detail/Chip-Resistor-Surface-Mount_100KR-1003-1_C14675.html" H 3200 4400 50  0001 C CNN "URL"
 	1    3200 4400
 	0    1    1    0
@@
 F 2 "Resistor_SMD:R_0603_1608Metric_Pad1.05x0.95mm_HandSolder" V 3630 3950 50  0001 C CNN
 F 3 "~" H 3700 3950 50  0001 C CNN
+F 4 "https://lcsc.com/product-detail/Chip-Resistor-Surface-Mount_100KR-1003-1_C14675.html" H 3700 3950 50  0001 C CNN "URL"
 	1    3700 3950
 	-1   0    0    1
@@
 F 2 "Package_TO_SOT_SMD:SOT-23_Handsoldering" H 4800 4250 50  0001 C CNN
 F 3 "~" H 4600 4150 50  0001 C CNN
+F 4 "https://lcsc.com/product-detail/MOSFET_Alpha-Omega-Semicon_AO3415_Alpha-Omega-Semicon-AOS-AO3415_C14354.html" H 4600 4150 50  0001 C CNN "URL"
 	1    4600 4150
 	1    0    0    1
@@
 F 0 "J22" H 5030 4492 50  0000 L CNN
 F 1 "Screw_Terminal_01x02" H 5030 4401 50  0000 L CNN
-F 2 "TerminalBlock:TerminalBlock_bornier-2_P5.08mm" H 4950 4500 50  0001 C CNN
+F 2 "Connector_PinHeader_2.54mm:PinHeader_1x02_P2.54mm_Vertical" H 4950 4500 50  0001 C CNN
 F 3 "~" H 4950 4500 50  0001 C CNN
 	1    4950 4500
@@
 F 2 "Package_TO_SOT_SMD:SOT-23_Handsoldering" H 8100 3300 50  0001 C CNN
 F 3 "~" H 7900 3200 50  0001 C CNN
+F 4 "https://lcsc.com/product-detail/MOSFET_ALLPOWER-ShenZhen-Quan-Li-Semiconductor-AP2300_C360338.html" H 7900 3200 50  0001 C CNN "URL"
 	1    7900 3200
 	1    0    0    1
@@
 F 2 "Resistor_SMD:R_0603_1608Metric_Pad1.05x0.95mm_HandSolder" V 7380 3200 50  0001 C CNN
 F 3 "~" H 7450 3200 50  0001 C CNN
+F 4 "https://lcsc.com/product-detail/New-Arrivals_SANYEAR-SY0603JN10KP_C380762.html" H 7450 3200 50  0001 C CNN "URL"
 	1    7450 3200
 	0    1    1    0
@@
 F 2 "Resistor_SMD:R_0603_1608Metric_Pad1.05x0.95mm_HandSolder" V 7580 3450 50  0001 C CNN
 F 3 "~" H 7650 3450 50  0001 C CNN
+F 4 "https://lcsc.com/product-detail/Chip-Resistor-Surface-Mount_UNI-ROYAL-Uniroyal-Elec-0603WAJ0105T5E_C26098.html" H 7650 3450 50  0001 C CNN "URL"
 	1    7650 3450
 	-1   0    0    1
@@
 F 0 "J23" H 8330 2342 50  0000 L CNN
 F 1 "Screw_Terminal_01x02" H 8330 2251 50  0000 L CNN
-F 2 "TerminalBlock:TerminalBlock_bornier-2_P5.08mm" H 8250 2350 50  0001 C CNN
+F 2 "Connector_PinHeader_2.54mm:PinHeader_1x02_P2.54mm_Vertical" H 8250 2350 50  0001 C CNN
 F 3 "~" H 8250 2350 50  0001 C CNN
 	1    8250 2350
@@
 F 2 "Package_TO_SOT_SMD:SOT-23_Handsoldering" H 8100 4900 50  0001 C CNN
 F 3 "~" H 7900 4800 50  0001 C CNN
+F 4 "https://lcsc.com/product-detail/MOSFET_ALLPOWER-ShenZhen-Quan-Li-Semiconductor-AP2300_C360338.html" H 7900 4800 50  0001 C CNN "URL"
 	1    7900 4800
 	1    0    0    1
@@
 F 2 "Resistor_SMD:R_0603_1608Metric_Pad1.05x0.95mm_HandSolder" V 7380 4800 50  0001 C CNN
 F 3 "~" H 7450 4800 50  0001 C CNN
+F 4 "https://lcsc.com/product-detail/New-Arrivals_SANYEAR-SY0603JN10KP_C380762.html" H 7450 4800 50  0001 C CNN "URL"
 	1    7450 4800
 	0    1    1    0
@@
 F 2 "Resistor_SMD:R_0603_1608Metric_Pad1.05x0.95mm_HandSolder" V 7580 5050 50  0001 C CNN
 F 3 "~" H 7650 5050 50  0001 C CNN
+F 4 "https://lcsc.com/product-detail/Chip-Resistor-Surface-Mount_UNI-ROYAL-Uniroyal-Elec-0603WAJ0105T5E_C26098.html" H 7650 5050 50  0001 C CNN "URL"
 	1    7650 5050
 	-1   0    0    1
@@
 F 0 "J24" H 8380 4242 50  0000 L CNN
 F 1 "Screw_Terminal_01x02" H 8380 4151 50  0000 L CNN
-F 2 "TerminalBlock:TerminalBlock_bornier-2_P5.08mm" H 8300 4250 50  0001 C CNN
+F 2 "Connector_PinHeader_2.54mm:PinHeader_1x02_P2.54mm_Vertical" H 8300 4250 50  0001 C CNN
 F 3 "~" H 8300 4250 50  0001 C CNN
 	1    8300 4250
@@
 F 2 "Resistor_SMD:R_1210_3225Metric" H 4750 2100 50  0001 L CNN
 F 3 "~" H 4700 2300 50  0001 C CNN
+F 4 "https://lcsc.com/product-detail/PTC-Resettable-Fuses_TECHFUSE-SL1210400_C70186.html" H 4700 2300 50  0001 C CNN "URL"
 	1    4700 2300
 	1    0    0    -1
@@
 F 2 "Resistor_SMD:R_1210_3225Metric" H 4750 3600 50  0001 L CNN
 F 3 "~" H 4700 3800 50  0001 C CNN
+F 4 "https://lcsc.com/product-detail/PTC-Resettable-Fuses_TECHFUSE-SL1210400_C70186.html" H 4700 3800 50  0001 C CNN "URL"
 	1    4700 3800
 	1    0    0    -1
@@
 F 2 "Resistor_SMD:R_1210_3225Metric" H 8050 4250 50  0001 L CNN
 F 3 "~" H 8000 4450 50  0001 C CNN
+F 4 "https://lcsc.com/product-detail/PTC-Resettable-Fuses_TECHFUSE-SL1210400_C70186.html" H 8000 4450 50  0001 C CNN "URL"
 	1    8000 4450
 	1    0    0    -1
@@
 F 2 "Resistor_SMD:R_1210_3225Metric" H 8050 2600 50  0001 L CNN
 F 3 "~" H 8000 2800 50  0001 C CNN
+F 4 "https://lcsc.com/product-detail/PTC-Resettable-Fuses_TECHFUSE-SL1210400_C70186.html" H 8000 2800 50  0001 C CNN "URL"
 	1    8000 2800
 	1    0    0    -1
@@
 F 2 "Package_TO_SOT_SMD:SOT-23_Handsoldering" H 3800 3000 50  0001 C CNN
 F 3 "~" H 3600 2900 50  0001 C CNN
+F 4 "https://lcsc.com/product-detail/Transistors-NPN-PNP_S8050_C181158.html" H 3600 2900 50  0001 C CNN "URL"
 	1    3600 2900
 	1    0    0    -1
@@
 F 2 "Package_TO_SOT_SMD:SOT-23_Handsoldering" H 3800 4500 50  0001 C CNN
 F 3 "~" H 3600 4400 50  0001 C CNN
+F 4 "https://lcsc.com/product-detail/Transistors-NPN-PNP_S8050_C181158.html" H 3600 4400 50  0001 C CNN "URL"
 	1    3600 4400
 	1    0    0    -1
