File: hardware/mainBoard/SDI12.sch (KiCad schematic (older format))
At the start: 2 parts, among them J20 Screw_Terminal_01x06, U20 TXB0104PW

Commit message: First working software
Parts:
- U20: URL (none) -> https://lcsc.com/product-detail/Level-Translators-Shifters_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
Changed lines of the file:
@@
 EESchema Schematic File Version 4
+LIBS:prockeckv2-cache
 EELAYER 30 0
 EELAYER END
@@
 F 2 "Package_SO:TSSOP-14_4.4x5mm_P0.65mm" H 5150 3150 50  0001 C CNN
 F 3 "http://www.ti.com/lit/ds/symlink/txb0104.pdf" H 5260 3995 50  0001 C CNN
+F 4 "https://lcsc.com/product-detail/Level-Translators-Shifters_Texas-Instruments-TXB0104PWR_C60708.html" H 5150 3900 50  0001 C CNN "URL"
 	1    5150 3900
 	1    0    0    -1
